Commit message: did wk2p2

File: src/hrwros_week2/urdf/hrwros_assignment2.xacro (robot description, xacro)
@@ -72,3 +72,20 @@
   </joint>
   <!-- Add your solution to assignment 2 here -->
+  <material name="green">
+    <color rgba="0 1 0 1"/>
+  </material>
+  <link name="green_sphere">
+    <visual>
+      <origin xyz="0 0 0.4" />
+      <geometry>
+        <sphere radius="0.4"/>
+      </geometry>
+      <material name="green"/>
+    </visual>
+  </link>
+  <joint name="green_sphere_joint" type="fixed">
+    <parent link="world"/>
+    <child link="green_sphere"/>
+    <origin xyz="5.75 -4.5 0"/>
+  </joint>
 </robot>
